Commit message: abc

File: iiwa_3finger_description/urdf/iiwa_3finger.urdf.xacro (robot description, xacro)
@@ -2,4 +2,5 @@
 <!-- Here we define the robot, we named it "iiwa14_3finger_gripper" -->
 <robot xmlns:xacro="http://www.ros.org/wiki/xacro" name="iiwa_3finger">
+<xacro:macro name="iiwa_3finger" params="prefix">
   <!-- Import Rviz colors -->
   <xacro:include filename="$(find iiwa_description)/urdf/materials.xacro" />
@@ -16,5 +17,4 @@
   If you don't want to have that you can define a basic world link (see commented lines)
   -->
-  <xacro:macro name="iiwa_3finger" params="prefix">
     <!--     <link name="world"/> -->
   <link name="world">
@@ -170,4 +170,4 @@
       <implicitSpringDamper>1</implicitSpringDamper>
     </gazebo>
-  </xacro:macro>
+</xacro:macro>
 </robot>

Commit message: a

File: iiwa_3finger_description/urdf/iiwa_3finger.urdf.xacro (robot description, xacro)
@@ -2,14 +2,12 @@
 <!-- Here we define the robot, we named it "iiwa14_3finger_gripper" -->
 <robot xmlns:xacro="http://www.ros.org/wiki/xacro" name="iiwa_3finger">
-<xacro:macro name="iiwa_3finger" params="prefix">
   <!-- Import Rviz colors -->
   <xacro:include filename="$(find iiwa_description)/urdf/materials.xacro" />
   <!--Import the iiwa14 macro -->
   <xacro:include filename="$(find iiwa_description)/urdf/iiwa14.xacro"/>
-  <!-- Import robotiq finger -->
-  <xacro:include filename="$(find iiwa_3finger)/iiwa_3finger_description/urdf/robotiq_finger.urdf.xacro"/>
   <!--  Arguments for the iiwa14 macro  -->
   <xacro:arg name="hardware_interface" default="PositionJointInterface"/>
   <xacro:arg name="robot_name" default="iiwa"/>
+  <xacro:arg name="prefix" default=""/>
   <!--  Define the origin of your 3D space
   Here we define a box lying at 0,0,0 with some dimensions, in reality our robot is place on top of a metal cart with those dimensions.
@@ -170,4 +168,3 @@
       <implicitSpringDamper>1</implicitSpringDamper>
     </gazebo>
-</xacro:macro>
 </robot>

Commit message: a

File: iiwa_3finger_description/urdf/iiwa_3finger.urdf.xacro (robot description, xacro)
@@ -9,5 +9,5 @@
   <xacro:arg name="hardware_interface" default="PositionJointInterface"/>
   <xacro:arg name="robot_name" default="iiwa"/>
-  <xacro:arg name="prefix" default=""/>
+  <!-- xacro:arg name="prefix" default=""/-->
   <!--  Define the origin of your 3D space
   Here we define a box lying at 0,0,0 with some dimensions, in reality our robot is place on top of a metal cart with those dimensions.
@@ -81,14 +81,14 @@
   <joint name="couling_joint" type="fixed">
     <parent link="coupling_link" />
-    <child link = "${prefix}palm" />
+    <child link = "palm" />
     <origin xyz="0.04 0.07 0.04" rpy="${PI/2} ${PI/2} ${PI/2}" />
   </joint>
     <!-- Insert the fingers -->
-    <xacro:robotiq_finger prefix="${prefix}finger_1_"/>
-    <xacro:robotiq_finger prefix="${prefix}finger_2_"/>
-    <xacro:robotiq_finger prefix="${prefix}finger_middle_"/>
+    <xacro:robotiq_finger prefix="finger_1_"/>
+    <xacro:robotiq_finger prefix="finger_2_"/>
+    <xacro:robotiq_finger prefix="finger_middle_"/>
       <!-- link list -->
       <!-- Link palm -->
-      <link name="${prefix}palm">
+      <link name="palm">
         <visual>
           <geometry>
@@ -124,5 +124,5 @@
         </inertial>
       </link>
-      <gazebo reference="${prefix}palm">
+      <gazebo reference="palm">
         <mu1>1.1</mu1>
         <mu2>1.1</mu2>
@@ -131,7 +131,7 @@
     <!-- Joint list -->
     <!-- Joint palm_finger_1_joint -->
-    <joint name="${prefix}palm_finger_1_joint" type="revolute">
-      <parent link="${prefix}palm"/>
-      <child link="${prefix}finger_1_link_0"/>
+    <joint name="palm_finger_1_joint" type="revolute">
+      <parent link="palm"/>
+      <child link="finger_1_link_0"/>
       <dynamics damping="1" friction="0" />
       <axis xyz="0 1 0"/>
@@ -140,11 +140,11 @@
       <limit lower="-0.2967" upper="0.2967" effort="60" velocity="-1"/>
     </joint>
-    <gazebo reference="${prefix}palm_finger_1_joint">
+    <gazebo reference="palm_finger_1_joint">
       <implicitSpringDamper>1</implicitSpringDamper>
     </gazebo>
     <!-- Joint palm_finger_2_joint -->
-    <joint name="${prefix}palm_finger_2_joint" type="revolute">
-      <parent link="${prefix}palm"/>
-      <child link="${prefix}finger_2_link_0"/>
+    <joint name="palm_finger_2_joint" type="revolute">
+      <parent link="palm"/>
+      <child link="finger_2_link_0"/>
       <dynamics damping="1" friction="0" />
       <axis xyz="0 1 0"/>
@@ -153,11 +153,11 @@
       <limit lower="-0.2967" upper="0.2967" effort="60" velocity="-1"/>
     </joint>
-    <gazebo reference="${prefix}palm_finger_2_joint">
+    <gazebo reference="palm_finger_2_joint">
       <implicitSpringDamper>1</implicitSpringDamper>
     </gazebo>
     <!-- Joint palm_finger_middle_joint -->
-    <joint name="${prefix}palm_finger_middle_joint" type="revolute">
-      <parent link="${prefix}palm"/>
-      <child link="${prefix}finger_middle_link_0"/>
+    <joint name="palm_finger_middle_joint" type="revolute">
+      <parent link="palm"/>
+      <child link="finger_middle_link_0"/>
       <dynamics damping="1" friction="0" />
       <axis xyz="0 1 0"/>
@@ -165,5 +165,5 @@
       <limit lower="0" upper="0" effort="60" velocity="-1"/>
     </joint>
-    <gazebo reference="${prefix}palm_finger_middle_joint">
+    <gazebo reference="palm_finger_middle_joint">
       <implicitSpringDamper>1</implicitSpringDamper>
     </gazebo>

Commit message: fake control

File: iiwa_3finger_description/urdf/iiwa_3finger.urdf.xacro (robot description, xacro)
@@ -60,5 +60,5 @@
           <mesh filename="package://iiwa_3finger_description/meshes/visual/coupling.STL" />
         </geometry>
-        <material name="Black">
+        <material name="Grey">
           <!--color rgba="0 1 0 1"/-->
         </material>
@@ -69,5 +69,5 @@
           <mesh filename="package://iiwa_3finger_description/meshes/visual/collision/coupling.STL" />
         </geometry>
-        <material name="Black">
+        <material name="Grey">
           <!--color rgba="0 1 1 1"/-->
         </material>

Commit message: a

File: iiwa_3finger_description/urdf/iiwa_3finger.urdf.xacro (robot description, xacro)
@@ -1,5 +1,5 @@
 <?xml version="1.0"?>
 <!-- Here we define the robot, we named it "iiwa14_3finger_gripper" -->
-<robot xmlns:xacro="http://www.ros.org/wiki/xacro" name="iiwa_3finger">
+<robot xmlns:xacro="http://www.ros.org/wiki/xacro">
   <!-- Import Rviz colors -->
   <xacro:include filename="$(find iiwa_description)/urdf/materials.xacro" />
@@ -16,4 +16,5 @@
   If you don't want to have that you can define a basic world link (see commented lines)
   -->
+  <xacro:macro name="iiwa_3finger" params="parent hardware_interface robot_name *origin">
     <!--     <link name="world"/> -->
   <link name="world">
@@ -169,3 +170,4 @@
       <implicitSpringDamper>1</implicitSpringDamper>
     </gazebo>
+    </xacro:macro>
 </robot>
